File: USB_ISOLATOR/USB_ISOLATOR.kicad_pcb (KiCad board)
At the start: 2 copper layers, 17 parts, among them J1 USB_A, J2 USB_A, J3 Conn_01x02, U1 ADUM4160, U2 EL814, U3 TBA1-0511E

Commit message: j
Parts:
- added C5: 10u, Capacitor_SMD:C_0805_2012Metric, F.Cu at (147.8, 111.8)
- added C6: 10u, Capacitor_SMD:C_0805_2012Metric, F.Cu at (136.6, 111.9)
- added D2: green, LED_SMD:LED_0805_2012Metric, F.Cu at (193.8, 86.8)
- added FB1: GZ2012D601TF, Inductor_SMD:L_0805_2012Metric_Pad1.05x1.20mm_HandSolder, F.Cu at (132.8, 111.9)
- added FB2: GZ2012D601TF, Inductor_SMD:L_0805_2012Metric_Pad1.05x1.20mm_HandSolder, F.Cu at (151.7, 112.0)
- added Q1: MMBT3904, Package_TO_SOT_SMD:SOT-23, F.Cu at (189.1, 87.7)
- added R10: 10k, Resistor_SMD:R_0603_1608Metric, F.Cu at (176.5, 97.5)
- added R11: 22, Resistor_SMD:R_0402_1005Metric_Pad0.72x0.64mm_HandSolder, F.Cu at (180.1, 91.6)
- added R8: 3k3, Resistor_SMD:R_0603_1608Metric, F.Cu at (176.5, 95.0)
- added R9: 22, Resistor_SMD:R_0402_1005Metric_Pad0.72x0.64mm_HandSolder, F.Cu at (180.1, 89.6)
- U3: value TBA1-0511E -> ~; footprint Converter_DCDC:Converter_DCDC_Murata_MEE1SxxxxSC_THT -> Z_mycustom_footprint_lib:SIP7_DCDC single
- moved J1 62.1 mm to (61.8, 47.6)
- moved J2 62.1 mm to (61.8, 64.9)
- moved J3 56.5 mm to (193.8, 94.9)
- moved R1 55.0 mm to (185.2, 74.4)
- moved C1 50.3 mm to (176.5, 79.9)
- moved C2 50.3 mm to (176.5, 82.4)
- moved C3 50.3 mm to (176.5, 84.9)
- moved C4 50.3 mm to (176.5, 87.4)
- moved R5 50.3 mm to (176.5, 89.9)
- moved R7 50.3 mm to (176.5, 92.4)
- moved R2 47.9 mm to (180.1, 81.6)
- moved R3 47.9 mm to (180.1, 83.6)
- moved R4 47.9 mm to (180.1, 85.6)
- moved R6 47.9 mm to (180.1, 87.6)
- moved U3 30.8 mm to (135.3, 114.6)
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Connections:
- J3 pad 2: unconnected-(J3-Pin_2-Pad2) -> /Command
- U1 pad 4: unconnected-(U1-PDEN-Pad4) -> Net-(U1-PDEN)
- U2 pad 1: unconnected-(U2-Pad1) -> /Command
- U3 pad 1: +5VA -> Net-(U3-Vin)

Commit message: t
Parts:
- removed J2: USB_A, Connector_USB:USB_A_Molex_67643_Horizontal
- added D1: green, LED_SMD:LED_0805_2012Metric, F.Cu at (157.3, 116.1)
- added D3: ZMMxx, Diode_SMD:D_MiniMELF, F.Cu at (155.1, 113.8)
- added D4: LED_Small, LED_SMD:LED_0805_2012Metric, F.Cu at (131.2, 95.1)
- added H1: MountingHole, MountingHole:MountingHole_3mm, F.Cu at (155.0, 96.0)
- added R12: 10k, Resistor_SMD:R_0603_1608Metric, F.Cu at (157.3, 112.8)
- added R13: 10k, Resistor_SMD:R_0603_1608Metric, F.Cu at (128.7, 98.1)
- added R15: 3k3, Resistor_SMD:R_0603_1608Metric, F.Cu at (134.4, 95.4)
- added U4: LMV321, Package_TO_SOT_SMD:SOT-23-5_HandSoldering, F.Cu at (132.0, 98.0)
- added U5: SRV05-4, Package_TO_SOT_SMD:SOT-23-6, F.Cu at (154.7, 106.4)
- added U6: SRV05-4, Package_TO_SOT_SMD:SOT-23-6, F.Cu at (129.7, 107.6)
- added U7: ~, Z_mycustom_footprint_lib:USB A male SMD, F.Cu at (162.5, 108.7)
- J3: footprint Connector_PinHeader_2.54mm:PinHeader_1x02_P2.54mm_Vertical -> Connector_PinHeader_2.54mm:PinHeader_1x03_P2.54mm_Vertical
- R11: value 22 -> 3k3; footprint Resistor_SMD:R_0402_1005Metric_Pad0.72x0.64mm_HandSolder -> Resistor_SMD:R_0603_1608Metric
- R5: value 10k -> 3k3
- moved J1 84.6 mm to (124.9, 103.9), turned to -90 degrees
- moved D2 67.9 mm to (132.0, 115.0), turned to 180 degrees
- moved J3 66.3 mm to (127.4, 94.5), turned to -90 degrees
- moved R1 62.2 mm to (133.0, 108.1)
- moved Q1 60.7 mm to (130.3, 102.8), turned to -90 degrees
- moved R2 53.5 mm to (133.0, 106.9)
- moved R10 50.0 mm to (129.5, 114.5), turned to -90 degrees
- moved R9 47.5 mm to (135.1, 104.5)
- moved C1 46.9 mm to (135.3, 102.4), turned to 90 degrees
- moved C2 46.8 mm to (133.7, 101.4), turned to -90 degrees
- moved R11 45.7 mm to (134.5, 93.9)
- moved R7 45.0 mm to (133.1, 104.5), turned to -90 degrees
- moved R5 41.9 mm to (135.4, 97.9), turned to -90 degrees
- moved R3 36.7 mm to (151.8, 106.9)
- moved R6 35.5 mm to (149.2, 105.1), turned to 90 degrees
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Connections:
- J1 pad 2: Net-(J1-D-) -> /D1-
- J1 pad 3: Net-(J1-D+) -> /D1+
- J3 pad 2: /Command -> Net-(J3-Pin_2)
- R1 pad 1: Net-(J1-D+) -> /D1+
- R1 pad 2: /D1+ -> /D3+
- R11 pad 2: Net-(Q1-B) -> Net-(R11-Pad2)
- R2 pad 1: Net-(J1-D-) -> /D1-
- R2 pad 2: /D1- -> /D3-
- R3 pad 1: /D2+ -> Net-(U1-DD+)
- R3 pad 2: Net-(J2-D+) -> /D2+
- R4 pad 1: /D2- -> Net-(U1-DD-)
- R4 pad 2: Net-(J2-D-) -> /D2-
- R5 pad 1: +3V3_2 -> /Command
- R5 pad 2: /SDP_2 -> Net-(Q1-B)
- R8 pad 1: +5VA -> +3V3_2
- R8 pad 2: /Command -> /SDP_2
- U1 pad 10: /D2+ -> Net-(U1-DD+)
- U1 pad 11: /D2- -> Net-(U1-DD-)
- U1 pad 6: /D1- -> /D3-
- U1 pad 7: /D1+ -> /D3+
- U2 pad 1: /Command -> Net-(R11-Pad2)
Routing:
- net +5VA: track 0.00 -> 36.7 mm, vias 0 -> 1
- net +5VL: track 0.00 -> 33.5 mm, vias 0 -> 3
- net /SDP_2: track 0.00 -> 16.8 mm, vias 0 -> 2
- net GND2: track 0.00 -> 16.5 mm, vias 0 -> 10
- net GND1: track 0.00 -> 15.0 mm, vias 0 -> 11
- net Net-(J3-Pin_2): track 0.00 -> 11.0 mm
- net /D1-: track 0.00 -> 8.99 mm
- net /D1+: track 0.00 -> 8.81 mm
- net /Command: track 0.00 -> 8.52 mm
- net /SDP_1: track 0.00 -> 8.11 mm
- net /D2+: track 0.00 -> 7.35 mm
- net /D2-: track 0.00 -> 7.14 mm
- net Net-(Q1-B): track 0.00 -> 6.61 mm, vias 0 -> 2
- net +3V3_1: track 0.00 -> 6.44 mm
- net +3V3_2: track 0.00 -> 5.44 mm
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- added copper zone on In1.Cu, net GND1
- added copper zone on In2.Cu, net GND1
- added copper zone on In1.Cu, net GND2
Other:
- board outline added: 45 x 29 mm
- copper layers 2 -> 4

Commit message: g
Parts:
- moved C5 0.33 mm to (147.9, 111.6)
- moved D2 0.33 mm to (131.7, 115.0)
- moved C6 0.30 mm to (136.6, 111.6)
- moved R10 0.30 mm to (129.2, 114.5)
- moved FB2 0.23 mm to (151.9, 111.7)
- moved FB1 0.23 mm to (132.8, 111.7)
- moved D1 0.13 mm to (157.4, 116.1)
- moved D3 0.10 mm to (155.2, 113.8)
Other:
- board text added: "HIGH"
- board text added: "LOW"
- board text added: "LOW SPEED USB"
- board text added: "SPEED"
Changed lines of the file:
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@@
 		(tags "capacitor")
 		(property "Reference" "C1"
-			(at 0 -1.43 -90)
+			(at 0 -1.43 270)
 			(layer "F.SilkS")
+			(hide yes)
 			(effects
 				(font
@@
 	(footprint "Capacitor_SMD:C_0805_2012Metric"
 		(layer "F.Cu")
-		(at 136.6012 111.9124)
+		(at 136.6012 111.6076)
 		(descr "Capacitor SMD 0805 (2012 Metric), square (rectangular) end terminal, IPC_7351 nominal, (Body size source: IPC-SM-782 page 76, https://www.pcb-3d.com/wordpress/wp-content/uploads/ipc-sm-782a_amendment_1_and_2.pdf, https://docs.google.com/spreadsheets/d/1BsfQQcO9C6DZCsRaXUlFlo91Tg2WpOkGARC1WS5S8t0/edit?usp=sharing), generated with kicad-footprint-generator")
 		(tags "capacitor")
 		(property "Reference" "C6"
-			(at 0 -1.68 0)
+			(at 2.7686 0.0762 0)
 			(layer "F.SilkS")
 			(effects
@@
 		(tags "SMD DIP DIL PDIP SMDIP 2.54mm 9.53mm 375mil")
 		(property "Reference" "U2"
-			(at 0 -3.6 0)
+			(at 7.1374 -2.032 0)
 			(layer "F.SilkS")
 			(effects
@@
 		(tags "SOT TO_SOT_SMD")
 		(property "Reference" "U6"
-			(at 0 -2.4 270)
+			(at -2.8956 -0.889 0)
 			(layer "F.SilkS")
 			(effects
@@
 		)
 		(property "Value" "SRV05-4"
-			(at 0 2.4 270)
+			(at 0 2.4 -90)
 			(layer "F.Fab")
 			(effects
@@
 		)
 		(fp_text user "${REFERENCE}"
-			(at 0 0 270)
+			(at 0 0 -90)
 			(layer "F.Fab")
 			(effects
@@
 		(tags "SOT TO_SOT_SMD")
 		(property "Reference" "U5"
-			(at 0 -2.4 270)
+			(at 2.8448 0.5842 0)
 			(layer "F.SilkS")
 			(effects
@@
 		)
 		(property "Value" "SRV05-4"
-			(at 0 2.4 270)
+			(at 0 2.4 -90)
 			(layer "F.Fab")
 			(effects
@@
 		)
 		(fp_text user "${REFERENCE}"
-			(at 0 0 270)
+			(at 0 0 -90)
 			(layer "F.Fab")
 			(effects
@@
 		(tags "SOIC SO")
 		(property "Reference" "U1"
-			(at 0 -6.1 0)
+			(at 6.9088 4.6736 0)
 			(layer "F.SilkS")
 			(effects
@@
 		(tags "Through hole pin header THT 1x03 2.54mm single row")
 		(property "Reference" "J3"
-			(at 0 -2.33 -90)
+			(at -1.1684 -2.682 0)
 			(layer "F.SilkS")
+			(hide yes)
 			(effects
 				(font
@@
 		(tags "capacitor")
 		(property "Reference" "C4"
-			(at 0 1.4478 -90)
+			(at 2.286 1.6764 0)
 			(layer "F.SilkS")
 			(effects
@@
 			(at 0 -1.43 0)
 			(layer "F.SilkS")
+			(hide yes)
 			(effects
 				(font
@@
 	(footprint "Capacitor_SMD:C_0805_2012Metric"
 		(layer "F.Cu")
-		(at 147.8534 111.9378 180)
+		(at 147.8788 111.6076 180)
 		(descr "Capacitor SMD 0805 (2012 Metric), square (rectangular) end terminal, IPC_7351 nominal, (Body size source: IPC-SM-782 page 76, https://www.pcb-3d.com/wordpress/wp-content/uploads/ipc-sm-782a_amendment_1_and_2.pdf, https://docs.google.com/spreadsheets/d/1BsfQQcO9C6DZCsRaXUlFlo91Tg2WpOkGARC1WS5S8t0/edit?usp=sharing), generated with kicad-footprint-generator")
 		(tags "capacitor")
 		(property "Reference" "C5"
-			(at 0 -1.68 180)
+			(at 2.54 0.0508 180)
 			(layer "F.SilkS")
 			(effects
@@
 		(tags "SOT TO_SOT_SMD")
 		(property "Reference" "Q1"
-			(at 0 -2.4 90)
+			(at 1.5217 -1.2954 180)
 			(layer "F.SilkS")
 			(effects
@@
 		(tags "resistor")
 		(property "Reference" "R13"
-			(at 0 -1.43 -90)
+			(at -1.905 -2.1844 0)
 			(layer "F.SilkS")
+			(hide yes)
 			(effects
 				(font
@@
 		(tags "resistor")
 		(property "Reference" "R7"
-			(at 0 -1.43 90)
+			(at 1.143 -1.6002 180)
 			(layer "F.SilkS")
+			(hide yes)
 			(effects
 				(font
@@
 	(footprint "Resistor_SMD:R_0603_1608Metric"
 		(layer "F.Cu")
-		(at 129.4892 114.4778 -90)
+		(at 129.1844 114.4778 -90)
 		(descr "Resistor SMD 0603 (1608 Metric), square (rectangular) end terminal, IPC_7351 nominal, (Body size source: IPC-SM-782 page 72, https://www.pcb-3d.com/wordpress/wp-content/uploads/ipc-sm-782a_amendment_1_and_2.pdf), generated with kicad-footprint-generator")
 		(tags "resistor")
 		(property "Reference" "R10"
-			(at 0 -1.43 90)
+			(at 0.8128 2.286 180)
 			(layer "F.SilkS")
 			(effects
@@
 		(tags "resistor")
 		(property "Reference" "R12"
-			(at 0 -1.43 90)
+			(at 0.8382 -2.3368 180)
 			(layer "F.SilkS")
 			(effects
@@
 		(tags "resistor")
 		(property "Reference" "R8"
-			(at 0 1.3462 -90)
+			(at -0.3556 1.6256 0)
 			(layer "F.SilkS")
 			(effects
@@
 		(tags "capacitor")
 		(property "Reference" "C2"
-			(at 0 -1.43 90)
+			(at -1.016 1.7272 180)
 			(layer "F.SilkS")
 			(effects
@@
 		(tags "resistor handsolder")
 		(property "Reference" "R1"
-			(at 0 -1.17 0)
+			(at 2.0828 0.127 0)
 			(layer "F.SilkS")
 			(effects
@@
 		(tags "resistor")
 		(property "Reference" "R5"
-			(at 0 -1.43 90)
+			(at 1.016 -1.651 0)
 			(layer "F.SilkS")
 			(effects
@@
 		(at 162.5092 108.6612 90)
 		(property "Reference" "U7"
-			(at 6 -9.1 90)
+			(at -5.1562 0.7874 0)
 			(unlocked yes)
 			(layer "F.SilkS")
@@
 		(tags "USB_A Female Connector receptacle")
 		(property "Reference" "J1"
-			(at 3.5 -3.19 90)
+			(at 13.2536 3.2518 180)
 			(layer "F.SilkS")
 			(effects
@@
 	(footprint "LED_SMD:LED_0805_2012Metric"
 		(layer "F.Cu")
-		(at 157.3022 116.078 90)
+		(at 157.4292 116.078 90)
 		(descr "LED SMD 0805 (2012 Metric), square (rectangular) end terminal, IPC_7351 nominal, (Body size source: https://docs.google.com/spreadsheets/d/1BsfQQcO9C6DZCsRaXUlFlo91Tg2WpOkGARC1WS5S8t0/edit?usp=sharing), generated with kicad-footprint-generator")
 		(tags "LED")
 		(property "Reference" "D1"
-			(at -0.2032 1.8288 -90)
+			(at -2.8194 0.0762 0)
 			(layer "F.SilkS")
 			(effects
@@
 	(footprint "Inductor_SMD:L_0805_2012Metric_Pad1.05x1.20mm_HandSolder"
 		(layer "F.Cu")
-		(at 132.7912 111.9124)
+		(at 132.7912 111.6838)
 		(descr "Inductor SMD 0805 (2012 Metric), square (rectangular) end terminal, IPC_7351 nominal with elongated pad for handsoldering. (Body size source: IPC-SM-782 page 80, https://www.pcb-3d.com/wordpress/wp-content/uploads/ipc-sm-782a_amendment_1_and_2.pdf), generated with kicad-footprint-generator")
 		(tags "inductor handsolder")
@@
 		(tags "SOT-23-5 hand-soldering")
 		(property "Reference" "U4"
-			(at 0 -2.9 180)
+			(at 2.1844 -2.3739 180)
 			(layer "F.SilkS")
 			(effects
@@
 	(footprint "Inductor_SMD:L_0805_2012Metric_Pad1.05x1.20mm_HandSolder"
 		(layer "F.Cu")
-		(at 151.8666 111.9632)
+		(at 151.892 111.7346)
 		(descr "Inductor SMD 0805 (2012 Metric), square (rectangular) end terminal, IPC_7351 nominal with elongated pad for handsoldering. (Body size source: IPC-SM-782 page 80, https://www.pcb-3d.com/wordpress/wp-content/uploads/ipc-sm-782a_amendment_1_and_2.pdf), generated with kicad-footprint-generator")
 		(tags "inductor handsolder")
 		(property "Reference" "FB2"
-			(at -3.3782 0.0508 0)
+			(at 0.0508 -1.5494 0)
 			(layer "F.SilkS")
 			(effects
@@
 		(tags "LED")
 		(property "Reference" "D4"
-			(at 0 -1.65 0)
+			(at 0.635 -1.65 0)
 			(layer "F.SilkS")
+			(hide yes)
 			(effects
 				(font
@@
 	(footprint "LED_SMD:LED_0805_2012Metric"
 		(layer "F.Cu")
-		(at 132.0038 114.9604 180)
+		(at 131.6736 114.9604 180)
 		(descr "LED SMD 0805 (2012 Metric), square (rectangular) end terminal, IPC_7351 nominal, (Body size source: https://docs.google.com/spreadsheets/d/1BsfQQcO9C6DZCsRaXUlFlo91Tg2WpOkGARC1WS5S8t0/edit?usp=sharing), generated with kicad-footprint-generator")
 		(tags "LED")
@@
 		(tags "mounting hole 3mm no annular")
 		(property "Reference" "H1"
-			(at 0 -4 0)
+			(at 4.7914 -0.0134 0)
 			(layer "F.SilkS")
 			(effects
@@
 		(tags "resistor handsolder")
 		(property "Reference" "R6"
-			(at 0 -1.17 -90)
+			(at -1.905 0 0)
 			(layer "F.SilkS")
 			(effects
@@
 			(at 0 -1.43 0)
 			(layer "F.SilkS")
+			(hide yes)
 			(effects
 				(font
@@
 		(at 136.2202 114.3)
 		(property "Reference" "U3"
-			(at 6.858 -3.048 0)
+			(at 18.8976 5.334 0)
 			(unlocked yes)
 			(layer "F.SilkS")
@@
 			(at 0 -1.17 0)
 			(layer "F.SilkS")
+			(hide yes)
 			(effects
 				(font
@@
 	(footprint "Diode_SMD:D_MiniMELF"
 		(layer "F.Cu")
-		(at 155.1432 113.8174 -90)
+		(at 155.2448 113.8174 -90)
 		(descr "Diode Mini-MELF (SOD-80)")
 		(tags "Diode Mini-MELF (SOD-80)")
 		(property "Reference" "D3"
-			(at 3.81 0.4826 90)
+			(at 3.7338 0.1016 180)
 			(layer "F.SilkS")
 			(effects
@@
 		(tags "resistor handsolder")
 		(property "Reference" "R2"
-			(at 0 -1.17 0)
+			(at 2.0574 0 0)
 			(layer "F.SilkS")
 			(effects
@@
 		(tags "capacitor")
 		(property "Reference" "C3"
-			(at 0 -1.43 270)
+			(at 1.2192 1.651 0)
 			(layer "F.SilkS")
 			(effects
@@
 		)
 		(property "Value" "220n"
-			(at 0 1.43 270)
+			(at 0 1.43 -90)
 			(layer "F.Fab")
 			(effects
@@
 		)
 		(fp_text user "${REFERENCE}"
-			(at 0 0 270)
+			(at 0 0 -90)
 			(layer "F.Fab")
 			(effects
@@
 		(layer "Edge.Cuts")
 	)
+	(gr_text "LOW SPEED USB"
+		(at 129.3114 93.091 0)
+		(layer "F.SilkS" knockout)
+		(effects
+			(font
+				(size 0.75 0.75)
+				(thickness 0.13)
+				(bold yes)
+			)
+			(justify left bottom)
+		)
+	)
+	(gr_text "LOW"
+		(at 124.6632 97.663 0)
+		(layer "F.SilkS" knockout)
+		(effects
+			(font
+				(size 1 1)
+				(thickness 0.2)
+				(bold yes)
+			)
+			(justify left bottom)
+		)
+	)
+	(gr_text "SPEED"
+		(at 122.9614 99.1616 0)
+		(layer "F.SilkS" knockout)
+		(effects
+			(font
+				(size 1 1)
+				(thickness 0.2)
+				(bold yes)
+			)
+			(justify left bottom)
+		)
+	)
+	(gr_text "HIGH"
+		(at 120.65 97.663 0)
+		(layer "F.SilkS" knockout)
+		(effects
+			(font
+				(size 1 1)
+				(thickness 0.2)
+				(bold yes)
+			)
+			(justify left bottom)
+		)
+	)
 	(segment

Commit message: g
Parts:
- moved H1 1.00 mm to (156.0, 96.0)
Connections:
- net Net-(U1-DD+) renamed /D4+
- net Net-(U1-DD-) renamed /D4-
Routing:
- net +5VA: track 36.7 -> 35.6 mm
Other:
- board text added: "COM"
Changed lines of the file:
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@@
 	(net 28 "unconnected-(U6-IO3-Pad4)")
 	(net 29 "unconnected-(U6-IO2-Pad3)")
-	(net 30 "Net-(U1-DD+)")
-	(net 31 "Net-(U1-DD-)")
+	(net 30 "/D4+")
+	(net 31 "/D4-")
 	(net 32 "/D3+")
 	(net 33 "/D3-")
@@
 		(tags "capacitor")
 		(property "Reference" "C1"
-			(at 0 -1.43 270)
+			(at 0 -1.43 -90)
 			(layer "F.SilkS")
 			(hide yes)
@@
 			(net 29 "unconnected-(U6-IO2-Pad3)")
 			(pinfunction "IO2")
-			(pintype "passive")
+			(pintype "passive+no_connect")
 		)
 		(pad "4" smd roundrect
@@
 			(net 28 "unconnected-(U6-IO3-Pad4)")
 			(pinfunction "IO3")
-			(pintype "passive")
+			(pintype "passive+no_connect")
 		)
 		(pad "5" smd roundrect
@@
 			(net 9 "unconnected-(U5-IO2-Pad3)")
 			(pinfunction "IO2")
-			(pintype "passive")
+			(pintype "passive+no_connect")
 		)
 		(pad "4" smd roundrect
@@
 			(net 10 "unconnected-(U5-IO3-Pad4)")
 			(pinfunction "IO3")
-			(pintype "passive")
+			(pintype "passive+no_connect")
 		)
 		(pad "5" smd roundrect
@@
 			(layers "F.Cu" "F.Paste" "F.Mask")
 			(roundrect_rratio 0.25)
-			(net 30 "Net-(U1-DD+)")
+			(net 30 "/D4+")
 			(pinfunction "DD+")
 			(pintype "bidirectional")
@@
 			(layers "F.Cu" "F.Paste" "F.Mask")
 			(roundrect_rratio 0.25)
-			(net 31 "Net-(U1-DD-)")
+			(net 31 "/D4-")
 			(pinfunction "DD-")
 			(pintype "bidirectional")
@@
 			(layers "F.Cu" "F.Paste" "F.Mask")
 			(roundrect_rratio 0.25)
-			(net 30 "Net-(U1-DD+)")
+			(net 30 "/D4+")
 			(pintype "passive")
 		)
@@
 			(layers "F.Cu" "F.Paste" "F.Mask")
 			(roundrect_rratio 0.25)
-			(net 31 "Net-(U1-DD-)")
+			(net 31 "/D4-")
 			(pintype "passive")
 		)
@@
 		(tags "inductor handsolder")
 		(property "Reference" "FB1"
-			(at -3.302 0.0254 0)
+			(at -0.889 1.5494 0)
 			(layer "F.SilkS")
 			(effects
@@
 	(footprint "MountingHole:MountingHole_3mm"
 		(layer "F.Cu")
-		(at 155 96)
+		(at 156 96)
 		(descr "Mounting Hole 3mm, no annular")
 		(tags "mounting hole 3mm no annular")
@@
 		(layer "Edge.Cuts")
 	)
+	(gr_text "COM"
+		(at 123.8504 92.964 0)
+		(layer "F.SilkS" knockout)
+		(effects
+			(font
+				(size 0.7 0.7)
+				(thickness 0.13)
+				(bold yes)
+			)
+			(justify left bottom)
+		)
+	)
 	(gr_text "LOW SPEED USB"
 		(at 129.3114 93.091 0)
@@
 	)
 	(segment
+		(start 128.6642 98.9452)
+		(end 128.7018 98.9452)
+		(width 0.3)
+		(layer "F.Cu")
+		(net 3)
+	)
+	(segment
 		(start 132.7912 100.5332)
 		(end 131.2149 98.9569)
@@
 	)
 	(segment
+		(start 128.0668 103.9166)
+		(end 128.0668 99.5426)
+		(width 0.3)
+		(layer "F.Cu")
+		(net 3)
+	)
+	(segment
 		(start 137.6408 100.5332)
 		(end 132.7912 100.5332)
@@
 	)
 	(segment
-		(start 129.9008 113.6528)
-		(end 131.6412 111.9124)
+		(start 129.1844 113.2332)
+		(end 130.5052 111.9124)
 		(width 0.3)
 		(layer "F.Cu")
@@
 	)
 	(segment
-		(start 128.0974 103.9166)
-		(end 127.635 103.9166)
+		(start 128.0668 99.5426)
+		(end 128.6642 98.9452)
 		(width 0.3)
 		(layer "F.Cu")
@@
 	)
 	(segment
-		(start 127.635 100.012)
-		(end 128.7018 98.9452)
+		(start 128.0974 103.9166)
+		(end 128.0668 103.9166)
 		(width 0.3)
 		(layer "F.Cu")
@@
 	)
 	(segment
-		(start 128.7135 98.9569)
-		(end 128.7018 98.9452)
+		(start 129.1844 113.348)
+		(end 129.1844 113.2332)
 		(width 0.3)
 		(layer "F.Cu")
@@
 	)
 	(segment
-		(start 127.635 103.9166)
-		(end 127.635 100.012)
+		(start 128.7135 98.9569)
+		(end 128.7018 98.9452)
 		(width 0.3)
 		(layer "F.Cu")
@@
 	(segment
 		(start 129.4892 113.6528)
-		(end 129.9008 113.6528)
+		(end 129.1844 113.348)
 		(width 0.3)
 		(layer "F.Cu")

Commit message: ,
Parts:
- added FID1: Fiducial, Symbol:OSHW-Logo2_9.8x8mm_SilkScreen, B.Cu at (133.5, 106.5)
- added FID2: Fiducial, Symbol:KiCad-Logo_5mm_SilkScreen, B.Cu at (157.4, 117.9)
- added G***: LOGO, LOGO, B.Cu at (154.2, 106.3)
- added J2: Conn_01x02, Connector_PinHeader_2.54mm:PinHeader_1x03_P2.54mm_Vertical, F.Cu at (125.7, 118.8)
- D3: value ZMMxx -> ZMM5V6-M
- moved R10 0.10 mm to (129.1, 114.5)
- moved D2 0.08 mm to (131.6, 115.0)
Connections:
- C2 pad 1: +5VA -> Net-(J2-Pin_2)
- U1 pad 1: +5VA -> Net-(J2-Pin_2)
Routing:
- net Net-(J2-Pin_2): track 0.00 -> 25.0 mm, vias 0 -> 1
- net +5VL: track 33.5 -> 31.9 mm
- net GND1: track 15.0 -> 13.8 mm, vias 11 -> 13
- net /D2-: track 7.14 -> 6.26 mm
- net +3V3_1: track 6.44 -> 5.60 mm
- net Net-(R11-Pad2): track 2.41 -> 1.62 mm
- net GND2: track 16.5 -> 15.7 mm, vias 10 -> 22
- net /D2+: track 7.35 -> 6.67 mm
- net +5VA: track 35.6 -> 36.3 mm
- added copper zone on In2.Cu, net GND2
Other:
- board text added: "DATA_ON"

Commit message: g
Parts:
- added J4: Y1 cap, Connector_PinHeader_2.54mm:PinHeader_1x01_P2.54mm_Vertical, F.Cu at (133.5, 109.8)
- added J5: Y1 cap, Connector_PinHeader_2.54mm:PinHeader_1x01_P2.54mm_Vertical, F.Cu at (151.1, 109.3)
- moved U7 0.41 mm to (162.1, 108.7)
- moved R1 0.15 mm to (133.0, 108.0)
- moved R2 0.08 mm to (133.0, 107.0)
- moved R12 0.08 mm to (157.3, 112.8)
Routing:
- net /D2-: track 6.26 -> 9.07 mm
- net /D2+: track 6.67 -> 9.20 mm
- net +5VL: track 31.9 -> 33.0 mm
