File: USB_ISOLATOR/USB_ISOLATOR.kicad_sch (KiCad schematic)
At the start: 18 parts, among them J1 USB_A, J2 USB_A, J3 Conn_01x02, SW1 MCU_RESET, U1 ADUM4160, U2 EL814, U3 TBA1-0511E

Commit message: j
Parts:
- removed SW1: MCU_RESET, SamacSys_Parts:PTS526SK15SMTR2LFS, symbol Switch:SW_SPST
- removed U3: TBA1-0511E, Converter_DCDC:Converter_DCDC_Murata_MEE1SxxxxSC_THT, symbol Converter_DCDC:TBA1-0511E
- added C5, C6: 10u, Capacitor_SMD:C_0805_2012Metric, symbol Device:C_Small
- added D1, D2: green, LED_SMD:LED_0805_2012Metric, symbol Device:LED_Small
- added FB1, FB2: GZ2012D601TF, Inductor_SMD:L_0805_2012Metric_Pad1.05x1.20mm_HandSolder, symbol Device:FerriteBead_Small
- added Q1: MMBT3904, Package_TO_SOT_SMD:SOT-23, symbol Transistor_BJT:MMBT3904
- added R10, R12: 10k, Resistor_SMD:R_0603_1608Metric, symbol Device:R_Small
- added R11, R9: 22, Resistor_SMD:R_0402_1005Metric_Pad0.72x0.64mm_HandSolder, symbol Device:R_Small
- added R8: 3k3, Resistor_SMD:R_0603_1608Metric, symbol Device:R_Small
- added U3: ~, Z_mycustom_footprint_lib:SIP7_DCDC single, symbol My_custom_lib:E_S-2WR3&F_S-2WR3
Connections:
- net +3V3_1: now also R9.1
- net +5VA: now also FB1.1, R10.1, R8.1
- net +5VL: now also FB2.2, R12.1
- net GND1: now also C6.2, D2.1 (K), Q1.2 (E), U3.2 (GND_1)
- net GND2: now also C5.2, D1.1 (K), U3.5 (GND_2)
- net SDP_1: now also Q1.3 (C)
- net Command: now reaches J3.2 (Pin_2)
- net Command: now also U2.1, R11.1, R8.2
- net at U1.4 (PDEN): now also R9.2
- new net: C5.1, FB2.1, U3.7 (Vout)
- new net: Q1.1 (B), R11.2
- new net: D1.2 (A), R12.2
- new net: D2.2 (A), R10.2
- new net: C6.1, FB1.2, U3.1 (Vin)
Other:
- moved on the sheet: C1, C2, C3, J1, J2, J3, R1, R2, R3, R4, R5, R7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

Commit message: t
Parts:
- removed J2: USB_A, Connector_USB:USB_A_Molex_67643_Horizontal, symbol Connector:USB_A
- added D3: ZMMxx, Diode_SMD:D_MiniMELF, symbol Diode:ZMMxx
- added D4: LED_Small, LED_SMD:LED_0805_2012Metric, symbol Device:LED_Small
- added H1: MountingHole, MountingHole:MountingHole_3mm, symbol Mechanical:MountingHole
- added R13: 10k, Resistor_SMD:R_0603_1608Metric, symbol Device:R_Small
- added R15: 3k3, Resistor_SMD:R_0603_1608Metric, symbol Device:R_Small
- added U4: LMV321, Package_TO_SOT_SMD:SOT-23-5_HandSoldering, symbol Amplifier_Operational:LMV321
- added U5, U6: SRV05-4, Package_TO_SOT_SMD:SOT-23-6, symbol Power_Protection:SRV05-4
- added U7: ~, Z_mycustom_footprint_lib:USB A male SMD, symbol My_custom_lib:USB_A_male
- J3: footprint Connector_PinHeader_2.54mm:PinHeader_1x02_P2.54mm_Vertical -> Connector_PinHeader_2.54mm:PinHeader_1x03_P2.54mm_Vertical
- R11: value 22 -> 3k3; footprint Resistor_SMD:R_0402_1005Metric_Pad0.72x0.64mm_HandSolder -> Resistor_SMD:R_0603_1608Metric; LCSC C25092 -> C22978
- R5: value 10k -> 3k3; LCSC C25804 -> C22978
Connections:
- net +3V3_2: now also R8.1; no longer R5.1
- net +5VA: now also R13.1, U4.5 (V+), U6.5 (VP); no longer R8.1
- net +5VL: now also D3.1 (K), U5.5 (VP), U7.1 (Vbus)
- net Command: now also R5.1, R15.2, U4.3 (-), U4.4; no longer J3.2 (Pin_2), R8.2, U2.1
- net D1+: now also J1.3 (D+), R1.1, U6.1 (IO1); no longer R1.2, U1.7 (UD+)
- net D1-: now also J1.2 (D-), R2.1, U6.6 (IO4); no longer R2.2, U1.6 (UD-)
- net D2+: now also R3.2, U5.1 (IO1), U7.3 (D+); no longer R3.1, U1.10 (DD+)
- net D2-: now also R4.2, U5.6 (IO4), U7.2 (D-); no longer R4.1, U1.11 (DD-)
- net GND1: now also D4.1 (K), U4.2 (V-), U6.2 (VN)
- net GND2: now also D3.2 (A), U5.2 (VN), U7.4 (GND)
- net SDP_2: now also R8.2; no longer R5.2
- net at Q1.1 (B): now also R5.2; no longer R11.2
- new net: J3.2 (Pin_2), R13.2, U4.1 (+)
- new net: R11.2, U2.1
- new net: R3.1, U1.10 (DD+)
- new net: R4.1, U1.11 (DD-)
- new net: D4.2 (A), R15.1
- new net D3+: R1.2, U1.7 (UD+)
- new net D3-: R2.2, U1.6 (UD-)
Other:
- moved on the sheet: C1, C2, C3, C4, C5, C6, D1, D2, FB1, FB2, J1, J3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

Commit message: g
Connections:
- net D4+: now reaches R3.1, U1.10 (DD+)
- net D4-: now reaches R4.1, U1.11 (DD-)
- no-connect marks 2 -> 6
Changed lines of the file:
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@@
+	)
+	(no_connect
+		(at 215.9 135.89)
 	)
 	(no_connect
@@
 		(at 118.11 97.79)
 	)
+	(no_connect
+		(at 241.3 130.81)
+	)
+	(no_connect
+		(at 40.64 76.2)
+	)
+	(no_connect
+		(at 66.04 71.12)
+	)
 	(wire
 		(pts
@@
 		)
 		(stroke
-			(width 0)
-			(type default)
+			(width 0.75)
+			(type dash)
 		)
 	)
@@
 		)
 	)
+	(label "D4-"
+		(at 193.04 90.17 0)
+		(fields_autoplaced yes)
+		(effects
+			(font
+				(size 1.27 1.27)
+			)
+			(justify left bottom)
+		)
+	)
 	(label "D2-"
 		(at 214.63 90.17 0)
@@
 		(fields_autoplaced yes)
 		(effects
+			(font
+				(size 1.27 1.27)
+			)
+			(justify left bottom)
+		)
+	)
+	(label "D4+"
+		(at 193.04 87.63 0)
+		(fields_autoplaced yes)
+		(effects

Commit message: ,
Parts:
- added FID1: Fiducial, Symbol:OSHW-Logo2_9.8x8mm_SilkScreen, symbol Mechanical:Fiducial
- added FID2: Fiducial, Symbol:KiCad-Logo_5mm_SilkScreen, symbol Mechanical:Fiducial
- added J2: Conn_01x02, Connector_PinHeader_2.54mm:PinHeader_1x03_P2.54mm_Vertical, symbol Connector_Generic:Conn_01x02
- D3: value ZMMxx -> ZMM5V6-M; LCSC (none) -> C8062
- U1: LCSC (none) -> C57791
- U2: LCSC (none) -> C32565
Connections:
- net +5VA: now also J2.1 (Pin_1); no longer C2.1, U1.1 (VBUS1)
- new net: C2.1, J2.2 (Pin_2), U1.1 (VBUS1)
Other:
- moved on the sheet: C2, D2, FB1, J1, R1, R10, R2

Commit message: g
Parts:
- added J4, J5: Y1 cap, Connector_PinHeader_2.54mm:PinHeader_1x01_P2.54mm_Vertical, symbol Connector:Conn_01x01_Pin
- U2: LCSC C32565 -> C106900
Connections:
- net GND1: now also J4.1 (Pin_1)
- net GND2: now also J5.1 (Pin_1)
